Commit message: car changes

File: assets/simplecar.urdf (robot description, URDF)
Before this commit: robot simplecar, 7 links, 6 joints
Links:
- link left_hinge: geometry visual box size=0.02 0.02 0.06
- link right_hinge: geometry visual box size=0.02 0.02 0.06
Joints:
- joint base_to_left_hinge: limit lower=-0.5 upper=0.5 effort=100 velocity=100 -> lower=-0.610865 upper=0.610865 effort=100 velocity=100; origin xyz=0.2 0.0 0 -> xyz=0.15 0.175 0
- joint base_to_right_hinge: limit lower=-0.5 upper=0.5 effort=100 velocity=100 -> lower=-0.610865 upper=0.610865 effort=100 velocity=100; origin xyz=0.2 0 0 -> xyz=0.15 -0.175 0
- joint left_hinge_to_left_front_wheel: origin xyz=0 0.2 0 -> xyz=0 0 0
- joint right_hinge_to_right_front_wheel: origin xyz=0 -0.2 0 -> xyz=0 0 0
